File: copyHHKB.sch (KiCad schematic (older format))
At the start: 130 parts, among them U1 ProMicro, U2 ProMicro, j1 SW_DIP_x01, k1 SW_DIP_x01, m1 SW_DIP_x01, p1 SW_DIP_x01, q1 SW_DIP_x01, t1 SW_DIP_x01, u1 SW_DIP_x01, x1 SW_DIP_x01, y1 SW_DIP_x01

Commit message: 作ってる
Parts:
- removed SW? (x2): SW_DIP_x01, symbol copyHHKB-rescue:SW_DIP_x01
- added s2, s3: sw, keyboard:TSHA-T-2.5B2-19E], symbol pin:sw
- !1, $1, %1, &1, '1, (1, )1, *1, +1, /1, ;1, <1, >1, @1, [1, ]1, ^1, _1, `1, a1, b1, c1, d1: footprint keebio:Kailh-PG1350-1u -> keyboard:MX_PCB_100H
- AltL1, AltR1: footprint keebio:Kailh-PG1350-1u -> keyboard:Hybrid_Plate_125H
- BackSP1: footprint keebio:Kailh-PG1350-1u -> keyboard:Hybrid_Plate_150H
- Control1, shiftR1: footprint keebio:Kailh-PG1350-1u -> keyboard:Hybrid_Plate_175H
- D1, D10, D11, D12, D13, D14, D15, D16, D17, D18, D19, D2, D20, D21, D22, D23, D24, D25, D26, D27, D28, D29, D3, D30, D31, D32, D33, D34, D35, D36, D37, D38, D39, D4, D40, D41, D42, D43, D44, D45, D46, D47, D48, D49, D5, D50, D51, D52, D53, D54, D55, D56, D57, D58, D59, D6, D60, D7, D8, D9: footprint keyboard:Diode -> keyboard:Diode-dual
- ESC1, Fn1, L1, e1, f1, g1, h1, i1, j1, k1, m1, n1, o1, p1, q1, r1, s1: footprint keebio:Kailh-PG1350-1u -> keyboard:Hybrid_PCB_100H
- Enter1: footprint keebio:Kailh-PG1350-1u -> keyboard:Hybrid_PCB_225H
- J1, J2: renamed from J?; footprint (none) -> SeparateHHKB:MJ-4PP-9_rev2
- SP1: footprint keebio:Kailh-PG1350-1u -> keyboard:MX_PCB_275H
- SP2: footprint keebio:Kailh-PG1350-1u -> keyboard:MX_Plate_225H
- U1, U2: footprint (none) -> pro micro:ProMicro
- p2, p3: renamed from p?; footprint (none) -> SeparateHHKB:StripLED_rev
- sharp1, t1, u1, v1, w1, winL1, winR1, x1, y1, z1, |1: footprint keebio:Kailh-PG1350-1u -> keyboard:MX_Plate_100H
- shiftL1: footprint keebio:Kailh-PG1350-1u -> keyboard:Hybrid_Plate_225H
- tab1: footprint keebio:Kailh-PG1350-1u -> keyboard:Hybrid_PCB_150H
Connections:
- wire segments 194 -> 196
- no-connect marks 11 -> 15
