File: SeparateHHKB.sch (KiCad schematic (older format))
At the start: 130 parts, among them J1 MJ-4PP-9, J2 MJ-4PP-9, U1 ProMicro, U2 ProMicro, j1 SW_DIP_x01, k1 SW_DIP_x01, m1 SW_DIP_x01, p1 SW_DIP_x01, p2 3pin, p3 3pin, q1 SW_DIP_x01, t1 SW_DIP_x01, u1 SW_DIP_x01, x1 SW_DIP_x01, y1 SW_DIP_x01

Commit message: 作ってる
Parts:
- AltL1, AltR1: footprint keyboard:Hybrid_Plate_125H -> keyboard:Hybrid_Plate_100H
- SP1: footprint keyboard:MX_Plate_100H -> keyboard:MX_PCB_275H
- SP2: footprint keyboard:MX_Plate_100H -> keyboard:MX_Plate_225H
- shiftR1: footprint keyboard:Hybrid_Plate_175H -> keyboard:Hybrid_Plate_275H
- winL1, winR1: footprint keyboard:MX_Plate_100H -> keyboard:MX_Plate_150H
Changed lines of the file:
@@
 EESchema Schematic File Version 4
-LIBS:copyHHKB-cache
+LIBS:SeparateHHKB-cache
 EELAYER 26 0
 EELAYER END
@@
 F 0 "shiftR1" H 12500 5350 50  0000 C CNN
 F 1 "SW_DIP_x01" H 12500 5050 50  0000 C CNN
-F 2 "keyboard:Hybrid_Plate_175H" H 12500 5200 50  0001 C CNN
+F 2 "keyboard:Hybrid_Plate_275H" H 12500 5200 50  0001 C CNN
 F 3 "" H 12500 5200 50  0001 C CNN
 	1    12500 5200
@@
 F 0 "AltL1" H -100 6050 50  0000 C CNN
 F 1 "SW_DIP_x01" H -100 5750 50  0000 C CNN
-F 2 "keyboard:Hybrid_Plate_125H" H -100 5900 50  0001 C CNN
+F 2 "keyboard:Hybrid_Plate_100H" H -100 5900 50  0001 C CNN
 F 3 "" H -100 5900 50  0001 C CNN
 	1    -100 5900
@@
 F 0 "AltR1" H 10700 6000 50  0000 C CNN
 F 1 "SW_DIP_x01" H 10700 5700 50  0000 C CNN
-F 2 "keyboard:Hybrid_Plate_125H" H 10700 5850 50  0001 C CNN
+F 2 "keyboard:Hybrid_Plate_100H" H 10700 5850 50  0001 C CNN
 F 3 "" H 10700 5850 50  0001 C CNN
 	1    10700 5850
@@
 F 0 "winL1" H 750 6050 50  0000 C CNN
 F 1 "SW_DIP_x01" H 750 5750 50  0000 C CNN
-F 2 "keyboard:MX_Plate_100H" H 750 5900 50  0001 C CNN
+F 2 "keyboard:MX_Plate_150H" H 750 5900 50  0001 C CNN
 F 3 "" H 750 5900 50  0001 C CNN
 	1    750  5900
@@
 F 0 "winR1" H 9850 6000 50  0000 C CNN
 F 1 "SW_DIP_x01" H 9850 5700 50  0000 C CNN
-F 2 "keyboard:MX_Plate_100H" H 9850 5850 50  0001 C CNN
+F 2 "keyboard:MX_Plate_150H" H 9850 5850 50  0001 C CNN
 F 3 "" H 9850 5850 50  0001 C CNN
 	1    9850 5850
@@
 F 0 "SP1" H 3300 6050 50  0000 C CNN
 F 1 "SW_DIP_x01" H 3300 5750 50  0000 C CNN
-F 2 "keyboard:MX_Plate_100H" H 3300 5900 50  0001 C CNN
+F 2 "keyboard:MX_PCB_275H" H 3300 5900 50  0001 C CNN
 F 3 "" H 3300 5900 50  0001 C CNN
 	1    3300 5900
@@
 F 0 "SP2" H 8150 6000 50  0000 C CNN
 F 1 "SW_DIP_x01" H 8150 5700 50  0000 C CNN
-F 2 "keyboard:MX_Plate_100H" H 8150 5850 50  0001 C CNN
+F 2 "keyboard:MX_Plate_225H" H 8150 5850 50  0001 C CNN
 F 3 "" H 8150 5850 50  0001 C CNN
 	1    8150 5850

Commit message: ちょっと前にスイッチの街がとかを修正したやつ
Parts:
- AltL1, AltR1: footprint keyboard:Hybrid_Plate_100H -> keyboard:MX_PCB_100H
- BackSP1: footprint keyboard:Hybrid_Plate_150H -> keyboard:MX_PCB_150H
- Control1: footprint keyboard:Hybrid_Plate_175H -> keyboard:MX_PCB_175H
- D61: footprint keyboard:Diode -> keyboard:Diode-dual
- ESC1, Fn1, L1, e1, f1, g1, h1, i1, j1, k1, m1, n1, o1, p1, q1, r1, s1: footprint keyboard:Hybrid_PCB_100H -> keyboard:MX_PCB_100H
- Enter1: footprint keyboard:Hybrid_PCB_225H -> keyboard:MX_PCB_225H
- SP2: footprint keyboard:MX_Plate_225H -> keyboard:MX_PCB_275H
- sharp1, t1, u1, v1, w1, x1, y1, z1, |1: footprint keyboard:MX_Plate_100H -> keyboard:MX_PCB_100H
- shiftL1: footprint keyboard:Hybrid_Plate_225H -> keyboard:MX_PCB_225H
- shiftR1: footprint keyboard:Hybrid_Plate_275H -> keyboard:MX_PCB_175H
- tab1: footprint keyboard:Hybrid_PCB_150H -> keyboard:MX_PCB_150H
- winL1, winR1: footprint keyboard:MX_Plate_150H -> keyboard:MX_PCB_100H
Changed lines of the file:
@@
 F 0 "ESC1" H -950 3850 50  0000 C CNN
 F 1 "SW_DIP_x01" H -950 3550 50  0000 C CNN
-F 2 "keyboard:Hybrid_PCB_100H" H -950 3700 50  0001 C CNN
+F 2 "keyboard:MX_PCB_100H" H -950 3700 50  0001 C CNN
 F 3 "" H -950 3700 50  0001 C CNN
 	1    -950 3700
@@
 F 0 "tab1" H -950 4350 50  0000 C CNN
 F 1 "SW_DIP_x01" H -950 4050 50  0000 C CNN
-F 2 "keyboard:Hybrid_PCB_150H" H -950 4200 50  0001 C CNN
+F 2 "keyboard:MX_PCB_150H" H -950 4200 50  0001 C CNN
 F 3 "" H -950 4200 50  0001 C CNN
 	1    -950 4200
@@
 F 0 "Control1" H -950 4850 50  0000 C CNN
 F 1 "SW_DIP_x01" H -950 4550 50  0000 C CNN
-F 2 "keyboard:Hybrid_Plate_175H" H -950 4700 50  0001 C CNN
+F 2 "keyboard:MX_PCB_175H" H -950 4700 50  0001 C CNN
 F 3 "" H -950 4700 50  0001 C CNN
 	1    -950 4700
@@
 F 0 "shiftL1" H -950 5350 50  0000 C CNN
 F 1 "SW_DIP_x01" H -950 5050 50  0000 C CNN
-F 2 "keyboard:Hybrid_Plate_225H" H -950 5200 50  0001 C CNN
+F 2 "keyboard:MX_PCB_225H" H -950 5200 50  0001 C CNN
 F 3 "" H -950 5200 50  0001 C CNN
 	1    -950 5200
@@
 F 0 "q1" H -100 4350 50  0000 C CNN
 F 1 "SW_DIP_x01" H -100 4050 50  0000 C CNN
-F 2 "keyboard:Hybrid_PCB_100H" H -100 4200 50  0001 C CNN
+F 2 "keyboard:MX_PCB_100H" H -100 4200 50  0001 C CNN
 F 3 "" H -100 4200 50  0001 C CNN
 	1    -100 4200
@@
 F 0 "z1" H 750 5400 50  0000 C CNN
 F 1 "SW_DIP_x01" H 750 5100 50  0000 C CNN
-F 2 "keyboard:MX_Plate_100H" H 750 5250 50  0001 C CNN
+F 2 "keyboard:MX_PCB_100H" H 750 5250 50  0001 C CNN
 F 3 "" H 750 5250 50  0001 C CNN
 	1    750  5250
@@
 F 0 "w1" H 750 4350 50  0000 C CNN
 F 1 "SW_DIP_x01" H 750 4050 50  0000 C CNN
-F 2 "keyboard:MX_Plate_100H" H 750 4200 50  0001 C CNN
+F 2 "keyboard:MX_PCB_100H" H 750 4200 50  0001 C CNN
 F 3 "" H 750 4200 50  0001 C CNN
 	1    750  4200
@@
 F 0 "s1" H 750 4850 50  0000 C CNN
 F 1 "SW_DIP_x01" H 750 4550 50  0000 C CNN
-F 2 "keyboard:Hybrid_PCB_100H" H 750 4700 50  0001 C CNN
+F 2 "keyboard:MX_PCB_100H" H 750 4700 50  0001 C CNN
 F 3 "" H 750 4700 50  0001 C CNN
 	1    750  4700
@@
 F 0 "x1" H 1600 5350 50  0000 C CNN
 F 1 "SW_DIP_x01" H 1600 5050 50  0000 C CNN
-F 2 "keyboard:MX_Plate_100H" H 1600 5200 50  0001 C CNN
+F 2 "keyboard:MX_PCB_100H" H 1600 5200 50  0001 C CNN
 F 3 "" H 1600 5200 50  0001 C CNN
 	1    1600 5200
@@
 F 0 "sharp1" H 1600 3850 50  0001 C CNN
 F 1 "SW_DIP_x01" H 1600 3550 50  0000 C CNN
-F 2 "keyboard:MX_Plate_100H" H 1600 3700 50  0001 C CNN
+F 2 "keyboard:MX_PCB_100H" H 1600 3700 50  0001 C CNN
 F 3 "" H 1600 3700 50  0001 C CNN
 	1    1600 3700
@@
 F 0 "e1" H 1600 4350 50  0000 C CNN
 F 1 "SW_DIP_x01" H 1600 4050 50  0000 C CNN
-F 2 "keyboard:Hybrid_PCB_100H" H 1600 4200 50  0001 C CNN
+F 2 "keyboard:MX_PCB_100H" H 1600 4200 50  0001 C CNN
 F 3 "" H 1600 4200 50  0001 C CNN
 	1    1600 4200
@@
 F 0 "r1" H 2450 4350 50  0000 C CNN
 F 1 "SW_DIP_x01" H 2450 4050 50  0000 C CNN
-F 2 "keyboard:Hybrid_PCB_100H" H 2450 4200 50  0001 C CNN
+F 2 "keyboard:MX_PCB_100H" H 2450 4200 50  0001 C CNN
 F 3 "" H 2450 4200 50  0001 C CNN
 	1    2450 4200
@@
 F 0 "f1" H 2450 4850 50  0000 C CNN
 F 1 "SW_DIP_x01" H 2450 4550 50  0000 C CNN
-F 2 "keyboard:Hybrid_PCB_100H" H 2450 4700 50  0001 C CNN
+F 2 "keyboard:MX_PCB_100H" H 2450 4700 50  0001 C CNN
 F 3 "" H 2450 4700 50  0001 C CNN
 	1    2450 4700
@@
 F 0 "v1" H 3300 5350 50  0000 C CNN
 F 1 "SW_DIP_x01" H 3300 5050 50  0000 C CNN
-F 2 "keyboard:MX_Plate_100H" H 3300 5200 50  0001 C CNN
+F 2 "keyboard:MX_PCB_100H" H 3300 5200 50  0001 C CNN
 F 3 "" H 3300 5200 50  0001 C CNN
 	1    3300 5200
@@
 F 0 "t1" H 3300 4350 50  0000 C CNN
 F 1 "SW_DIP_x01" H 3300 4050 50  0000 C CNN
-F 2 "keyboard:MX_Plate_100H" H 3300 4200 50  0001 C CNN
+F 2 "keyboard:MX_PCB_100H" H 3300 4200 50  0001 C CNN
 F 3 "" H 3300 4200 50  0001 C CNN
 	1    3300 4200
@@
 F 0 "g1" H 3300 4850 50  0000 C CNN
 F 1 "SW_DIP_x01" H 3300 4550 50  0000 C CNN
-F 2 "keyboard:Hybrid_PCB_100H" H 3300 4700 50  0001 C CNN
+F 2 "keyboard:MX_PCB_100H" H 3300 4700 50  0001 C CNN
 F 3 "" H 3300 4700 50  0001 C CNN
 	1    3300 4700
@@
 F 0 "y1" H 6450 4350 50  0000 C CNN
 F 1 "SW_DIP_x01" H 6450 4050 50  0000 C CNN
-F 2 "keyboard:MX_Plate_100H" H 6450 4200 50  0001 C CNN
+F 2 "keyboard:MX_PCB_100H" H 6450 4200 50  0001 C CNN
 F 3 "" H 6450 4200 50  0001 C CNN
 	1    6450 4200
@@
 F 0 "h1" H 6450 4850 50  0000 C CNN
 F 1 "SW_DIP_x01" H 6450 4550 50  0000 C CNN
-F 2 "keyboard:Hybrid_PCB_100H" H 6450 4700 50  0001 C CNN
+F 2 "keyboard:MX_PCB_100H" H 6450 4700 50  0001 C CNN
 F 3 "" H 6450 4700 50  0001 C CNN
 	1    6450 4700
@@
 F 0 "n1" H 7300 5350 50  0000 C CNN
 F 1 "SW_DIP_x01" H 7300 5050 50  0000 C CNN
-F 2 "keyboard:Hybrid_PCB_100H" H 7300 5200 50  0001 C CNN
+F 2 "keyboard:MX_PCB_100H" H 7300 5200 50  0001 C CNN
 F 3 "" H 7300 5200 50  0001 C CNN
 	1    7300 5200
@@
 F 0 "u1" H 7300 4350 50  0000 C CNN
 F 1 "SW_DIP_x01" H 7300 4050 50  0000 C CNN
-F 2 "keyboard:MX_Plate_100H" H 7300 4200 50  0001 C CNN
+F 2 "keyboard:MX_PCB_100H" H 7300 4200 50  0001 C CNN
 F 3 "" H 7300 4200 50  0001 C CNN
 	1    7300 4200
@@
 F 0 "j1" H 7300 4850 50  0000 C CNN
 F 1 "SW_DIP_x01" H 7300 4550 50  0000 C CNN
-F 2 "keyboard:Hybrid_PCB_100H" H 7300 4700 50  0001 C CNN
+F 2 "keyboard:MX_PCB_100H" H 7300 4700 50  0001 C CNN
 F 3 "" H 7300 4700 50  0001 C CNN
 	1    7300 4700
@@
 F 0 "m1" H 8150 5350 50  0000 C CNN
 F 1 "SW_DIP_x01" H 8150 5050 50  0000 C CNN
-F 2 "keyboard:Hybrid_PCB_100H" H 8150 5200 50  0001 C CNN
+F 2 "keyboard:MX_PCB_100H" H 8150 5200 50  0001 C CNN
 F 3 "" H 8150 5200 50  0001 C CNN
 	1    8150 5200
@@
 F 0 "i1" H 8150 4350 50  0000 C CNN
 F 1 "SW_DIP_x01" H 8150 4050 50  0000 C CNN
-F 2 "keyboard:Hybrid_PCB_100H" H 8150 4200 50  0001 C CNN
+F 2 "keyboard:MX_PCB_100H" H 8150 4200 50  0001 C CNN
 F 3 "" H 8150 4200 50  0001 C CNN
 	1    8150 4200
@@
 F 0 "k1" H 8150 4850 50  0000 C CNN
 F 1 "SW_DIP_x01" H 8150 4550 50  0000 C CNN
-F 2 "keyboard:Hybrid_PCB_100H" H 8150 4700 50  0001 C CNN
+F 2 "keyboard:MX_PCB_100H" H 8150 4700 50  0001 C CNN
 F 3 "" H 8150 4700 50  0001 C CNN
 	1    8150 4700
@@
 F 0 "o1" H 9000 4350 50  0000 C CNN
 F 1 "SW_DIP_x01" H 9000 4050 50  0000 C CNN
-F 2 "keyboard:Hybrid_PCB_100H" H 9000 4200 50  0001 C CNN
+F 2 "keyboard:MX_PCB_100H" H 9000 4200 50  0001 C CNN
 F 3 "" H 9000 4200 50  0001 C CNN
 	1    9000 4200
@@
 F 0 "L1" H 9000 4850 50  0000 C CNN
 F 1 "SW_DIP_x01" H 9000 4550 50  0000 C CNN
-F 2 "keyboard:Hybrid_PCB_100H" H 9000 4700 50  0001 C CNN
+F 2 "keyboard:MX_PCB_100H" H 9000 4700 50  0001 C CNN
 F 3 "" H 9000 4700 50  0001 C CNN
 	1    9000 4700
@@
 F 0 "p1" H 9850 4350 50  0000 C CNN
 F 1 "SW_DIP_x01" H 9850 4050 50  0000 C CNN
-F 2 "keyboard:Hybrid_PCB_100H" H 9850 4200 50  0001 C CNN
+F 2 "keyboard:MX_PCB_100H" H 9850 4200 50  0001 C CNN
 F 3 "" H 9850 4200 50  0001 C CNN
 	1    9850 4200
@@
 F 0 "shiftR1" H 12500 5350 50  0000 C CNN
 F 1 "SW_DIP_x01" H 12500 5050 50  0000 C CNN
-F 2 "keyboard:Hybrid_Plate_275H" H 12500 5200 50  0001 C CNN
+F 2 "keyboard:MX_PCB_175H" H 12500 5200 50  0001 C CNN
 F 3 "" H 12500 5200 50  0001 C CNN
 	1    12500 5200
@@
 F 0 "|1" H 12500 3850 50  0000 C CNN
 F 1 "SW_DIP_x01" H 12500 3550 50  0000 C CNN
-F 2 "keyboard:MX_Plate_100H" H 12500 3700 50  0001 C CNN
+F 2 "keyboard:MX_PCB_100H" H 12500 3700 50  0001 C CNN
 F 3 "" H 12500 3700 50  0001 C CNN
 	1    12500 3700
@@
 F 0 "BackSP1" H 12500 4350 50  0000 C CNN
 F 1 "SW_DIP_x01" H 12500 4050 50  0000 C CNN
-F 2 "keyboard:Hybrid_Plate_150H" H 12500 4200 50  0001 C CNN
+F 2 "keyboard:MX_PCB_150H" H 12500 4200 50  0001 C CNN
 F 3 "" H 12500 4200 50  0001 C CNN
 	1    12500 4200
@@
 F 0 "Enter1" H 12500 4850 50  0000 C CNN
 F 1 "SW_DIP_x01" H 12500 4550 50  0000 C CNN
-F 2 "keyboard:Hybrid_PCB_225H" H 12500 4700 50  0001 C CNN
+F 2 "keyboard:MX_PCB_225H" H 12500 4700 50  0001 C CNN
 F 3 "" H 12500 4700 50  0001 C CNN
 	1    12500 4700
@@
 F 0 "Fn1" H 11550 5350 50  0000 C CNN
 F 1 "SW_DIP_x01" H 11550 5050 50  0000 C CNN
-F 2 "keyboard:Hybrid_PCB_100H" H 11550 5200 50  0001 C CNN
+F 2 "keyboard:MX_PCB_100H" H 11550 5200 50  0001 C CNN
 F 3 "" H 11550 5200 50  0001 C CNN
 	1    11550 5200
@@
 F 0 "AltL1" H -100 6050 50  0000 C CNN
 F 1 "SW_DIP_x01" H -100 5750 50  0000 C CNN
-F 2 "keyboard:Hybrid_Plate_100H" H -100 5900 50  0001 C CNN
+F 2 "keyboard:MX_PCB_100H" H -100 5900 50  0001 C CNN
 F 3 "" H -100 5900 50  0001 C CNN
 	1    -100 5900
@@
 F 0 "AltR1" H 10700 6000 50  0000 C CNN
 F 1 "SW_DIP_x01" H 10700 5700 50  0000 C CNN
-F 2 "keyboard:Hybrid_Plate_100H" H 10700 5850 50  0001 C CNN
+F 2 "keyboard:MX_PCB_100H" H 10700 5850 50  0001 C CNN
 F 3 "" H 10700 5850 50  0001 C CNN
 	1    10700 5850
@@
 F 0 "winL1" H 750 6050 50  0000 C CNN
 F 1 "SW_DIP_x01" H 750 5750 50  0000 C CNN
-F 2 "keyboard:MX_Plate_150H" H 750 5900 50  0001 C CNN
+F 2 "keyboard:MX_PCB_100H" H 750 5900 50  0001 C CNN
 F 3 "" H 750 5900 50  0001 C CNN
 	1    750  5900
@@
 F 0 "winR1" H 9850 6000 50  0000 C CNN
 F 1 "SW_DIP_x01" H 9850 5700 50  0000 C CNN
-F 2 "keyboard:MX_Plate_150H" H 9850 5850 50  0001 C CNN
+F 2 "keyboard:MX_PCB_100H" H 9850 5850 50  0001 C CNN
 F 3 "" H 9850 5850 50  0001 C CNN
 	1    9850 5850
@@
 F 0 "SP2" H 8150 6000 50  0000 C CNN
 F 1 "SW_DIP_x01" H 8150 5700 50  0000 C CNN
-F 2 "keyboard:MX_Plate_225H" H 8150 5850 50  0001 C CNN
+F 2 "keyboard:MX_PCB_275H" H 8150 5850 50  0001 C CNN
 F 3 "" H 8150 5850 50  0001 C CNN
 	1    8150 5850
@@
 F 0 "D61" H 8450 6200 50  0000 C CNN
 F 1 "D" H 8450 6000 50  0000 C CNN
-F 2 "keyboard:Diode" H 8450 6100 50  0001 C CNN
+F 2 "keyboard:Diode-dual" H 8450 6100 50  0001 C CNN
 F 3 "" H 8450 6100 50  0001 C CNN
 	1    8450 6100
