File: copyHHKB.kicad_pcb (KiCad board)
At the start: 2 copper layers, 125 parts, among them U1 ARDUINO_MICRO_SHIELD, j1 SW_DIP_x01, k1 SW_DIP_x01, m1 SW_DIP_x01, p1 SW_DIP_x01, q1 SW_DIP_x01, t1 SW_DIP_x01, u1 SW_DIP_x01, x1 SW_DIP_x01, y1 SW_DIP_x01

Commit message: 作ってる
Parts:
- removed REF** (x3): MountingHole_3.2mm_M3, Mounting_Holes:MountingHole_3.2mm_M3
- removed a2, a3: SW_DIP_x01, keebio:Kailh-PG1350-1u
- added D61: D, keyboard:Diode, F.Cu at (130.0, 221.4)
- added J1: MJ-4PP-9, SeparateHHKB:MJ-4PP-9_rev2, F.Cu at (110.9, -2.19)
- added J2: MJ-4PP-9, SeparateHHKB:MJ-4PP-9_rev2, F.Cu at (118.8, -2.19)
- added SP2: SW_DIP_x01, keyboard:MX_Plate_225H, F.Cu at (190.5, 145.3)
- added U2: ProMicro, pro micro:ProMicro, F.Cu at (125.0, 211.2)
- added p2: 3pin, SeparateHHKB:StripLED_rev, F.Cu at (131.0, -1.68)
- added p3: 3pin, SeparateHHKB:StripLED_rev, F.Cu at (131.0, 4.92)
- added s2: sw, keyboard:TSHA-T-2.5B2-19E], F.Cu at (126.1, 0.74)
- added s3: sw, keyboard:TSHA-T-2.5B2-19E], F.Cu at (126.1, 7.09)
- added sharp1: SW_DIP_x01, keyboard:MX_Plate_100H, F.Cu at (-4.06, 53.3)
- !1, $1, %1, &1, '1, (1, )1, *1, +1, /1, ;1, <1, >1, @1, [1, ]1, ^1, _1, `1, a1, b1, c1, d1: footprint keebio:Kailh-PG1350-1u -> keyboard:MX_PCB_100H
- AltL1, AltR1: footprint keebio:Kailh-PG1350-1u -> keyboard:Hybrid_Plate_125H
- BackSP1: footprint keebio:Kailh-PG1350-1u -> keyboard:Hybrid_Plate_150H
- Control1: footprint keebio:Kailh-PG1350-1u -> keyboard:Hybrid_Plate_175H
- D1, D10, D11, D12, D13, D14, D15, D16, D17, D18, D19, D2, D20, D21, D22, D23, D24, D25, D26, D27, D28, D29, D3, D30, D31, D32, D33, D34, D35, D36, D37, D38, D39, D4, D40, D41, D42, D43, D44, D45, D46, D47, D48, D49, D5, D50, D51, D52, D53, D54, D55, D56, D57, D58, D59, D6, D60, D7, D8, D9: footprint keyboard:Diode -> keyboard:Diode-dual
- ESC1, Fn1, L1, e1, f1, g1, h1, i1, j1, k1, m1, n1, o1, p1, q1, r1, s1: footprint keebio:Kailh-PG1350-1u -> keyboard:Hybrid_PCB_100H
- Enter1: footprint keebio:Kailh-PG1350-1u -> keyboard:Hybrid_PCB_225H
- SP1: footprint keebio:Kailh-PG1350-1u -> keyboard:MX_PCB_275H
- U1: value ARDUINO_MICRO_SHIELD -> ProMicro; footprint micro:ARDUINO_MICRO_SHIELD -> pro micro:ProMicro
- shiftL1: footprint keebio:Kailh-PG1350-1u -> keyboard:Hybrid_Plate_225H
- shiftR1: footprint keebio:Kailh-PG1350-1u -> keyboard:Hybrid_Plate_275H
- t1, u1, v1, w1, x1, y1, z1, |1: footprint keebio:Kailh-PG1350-1u -> keyboard:MX_Plate_100H
- tab1: footprint keebio:Kailh-PG1350-1u -> keyboard:Hybrid_PCB_150H
- winL1, winR1: footprint keebio:Kailh-PG1350-1u -> keyboard:MX_Plate_150H
- moved SP1 102.7 mm to (24.4, 130.0)
- moved AltL1 68.2 mm to (-34.5, 130.3)
- moved Control1 68.2 mm to (-55.4, 91.4)
- moved D1 68.2 mm to (-71.1, 57.1)
- moved D11 68.2 mm to (-19.3, 93.5)
- moved D12 68.2 mm to (-9.40, 114.3)
- moved D13 68.2 mm to (-14.0, 57.1)
- moved D15 68.2 mm to (0.51, 93.5)
- moved D16 68.2 mm to (9.65, 114.3)
- moved D17 68.2 mm to (5.08, 57.1)
- moved D19 68.2 mm to (18.8, 93.5)
- moved D2 68.2 mm to (-65.8, 75.9)
- moved D20 68.2 mm to (28.7, 114.3)
- moved D21 68.2 mm to (24.1, 57.1)
- moved D23 68.2 mm to (37.8, 93.5)
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Connections:
- !1 pad 1: col1 -> Rcol1
- $1 pad 1: col4 -> Rcol4
- %1 pad 1: col5 -> Rcol5
- &1 pad 1: col7 -> Lcol7
- '1 pad 1: col11 -> Lcol11
- (1 pad 1: col9 -> Lcol9
- )1 pad 1: col10 -> Lcol10
- *1 pad 1: col8 -> Lcol8
- +1 pad 1: col12 -> Lcol12
- /1 pad 1: col11 -> Lcol11
- ;1 pad 1: col10 -> Lcol10
- <1 pad 1: col9 -> Lcol9
- >1 pad 1: col10 -> Lcol10
- @1 pad 1: col2 -> Rcol2
- AltL1 pad 1: col1 -> Rcol1
- AltR1 pad 1: col11 -> Lcol11
- BackSP1 pad 1: col13 -> Lcol13
- Control1 pad 1: col0 -> Rcol0
- D1 pad 1: row0 -> Rrow0
- D10 pad 1: row1 -> Rrow1
- D11 pad 1: row2 -> Rrow2
- D12 pad 1: row3 -> Rrow3
- D13 pad 1: row4 -> Rrow4
- D14 pad 1: row0 -> Rrow0
- D15 pad 1: row1 -> Rrow1
- D16 pad 1: row2 -> Rrow2
- D17 pad 1: row3 -> Rrow3
- D18 pad 1: row0 -> Rrow0
- D19 pad 1: row1 -> Rrow1
- D2 pad 1: row1 -> Rrow1
- D20 pad 1: row2 -> Rrow2
- D21 pad 1: row3 -> Rrow3
- D22 pad 1: row0 -> Rrow0
- D23 pad 1: row1 -> Rrow1
- D24 pad 1: row2 -> Rrow2
- D25 pad 1: row3 -> Rrow3
- D26 pad 1: row4 -> Rrow4
- D27 pad 1: row3 -> Rrow3
- D28 pad 1: row0 -> Lrow0
- D29 pad 1: row1 -> Lrow1
- D3 pad 1: row2 -> Rrow2
- D30 pad 1: row2 -> Lrow2
- D31 pad 1: row0 -> Lrow0
- D32 pad 1: row1 -> Lrow1
- D33 pad 1: row2 -> Lrow2
- D34 pad 1: row3 -> Lrow3
- D35 pad 1: row0 -> Lrow0
- D36 pad 1: row1 -> Lrow1
- D37 pad 1: row2 -> Lrow2
- D38 pad 1: row3 -> Lrow3
- D39 pad 1: row0 -> Lrow0
- D4 pad 1: row3 -> Rrow3
- D40 pad 1: row1 -> Lrow1
- D41 pad 1: row2 -> Lrow2
- D42 pad 1: row3 -> Lrow3
- D43 pad 1: row4 -> Lrow4
- D44 pad 1: row0 -> Lrow0
- D45 pad 1: row1 -> Lrow1
- D46 pad 1: row2 -> Lrow2
- D47 pad 1: row3 -> Lrow3
- D48 pad 1: row4 -> Lrow4
- D49 pad 1: row0 -> Lrow0
- D5 pad 1: row0 -> Rrow0
- D50 pad 1: row1 -> Lrow1
- D51 pad 1: row2 -> Lrow2
- D52 pad 1: row3 -> Lrow3
- D53 pad 1: row4 -> Lrow4
- D54 pad 1: row0 -> Lrow0
- D55 pad 1: row1 -> Lrow1
- D56 pad 1: row3 -> Lrow3
- D57 pad 1: row0 -> Lrow0
- D58 pad 1: row1 -> Lrow1
- D59 pad 1: row2 -> Lrow2
- D6 pad 1: row1 -> Rrow1
- D60 pad 1: row3 -> Lrow3
- D7 pad 1: row2 -> Rrow2
- D8 pad 1: row4 -> Rrow4
- D9 pad 1: row0 -> Rrow0
- ESC1 pad 1: col0 -> Rcol0
- Enter1 pad 1: col13 -> Lcol13
- Fn1 pad 1: col12 -> Lcol12
- L1 pad 1: col9 -> Lcol9
- SP1 pad 1: col5 -> Rcol5
- U1 pad 10: row4 -> Rrow3
- U1 pad 11: col5 -> Rrow4
- U1 pad 12: col12 -> (no net)
- U1 pad 13: col3 -> (no net)
- U1 pad 2: row1 -> Rdate
- U1 pad 3: row0 -> RGND
- U1 pad 4: col6 -> RGND
- U1 pad 5: col4 -> (no net)
- U1 pad 6: col11 -> (no net)
- U1 pad 7: col2 -> Rrow0
- U1 pad 8: col10 -> Rrow1
- U1 pad 9: col9 -> Rrow2
- [1 pad 1: col11 -> Lcol11
- ]1 pad 1: col12 -> Lcol12
- ^1 pad 1: col6 -> Lcol6
- _1 pad 1: col11 -> Lcol11
- `1 pad 1: col9 -> Lcol9
- a1 pad 1: col1 -> Rcol1
- b1 pad 1: col6 -> Rcol6
- c1 pad 1: col4 -> Rcol4
- d1 pad 1: col3 -> Rcol3
- e1 pad 1: col3 -> Rcol3
- f1 pad 1: col4 -> Rcol4
- g1 pad 1: col5 -> Rcol5
- h1 pad 1: col6 -> Lcol6
- i1 pad 1: col8 -> Lcol8
- j1 pad 1: col7 -> Lcol7
- k1 pad 1: col8 -> Lcol8
- m1 pad 1: col8 -> Lcol8
- n1 pad 1: col7 -> Lcol7
- o1 pad 1: col9 -> Lcol9
- p1 pad 1: col10 -> Lcol10
- q1 pad 1: col1 -> Rcol1
- r1 pad 1: col4 -> Rcol4
- s1 pad 1: col2 -> Rcol2
- shiftL1 pad 1: col0 -> Rcol0
- shiftR1 pad 1: col13 -> Lcol13
- t1 pad 1: col5 -> Rcol5
- tab1 pad 1: col0 -> Rcol0
- u1 pad 1: col7 -> Lcol7
- v1 pad 1: col5 -> Rcol5
- w1 pad 1: col2 -> Rcol2
- winL1 pad 1: col2 -> Rcol2
- winR1 pad 1: col10 -> Lcol10
- x1 pad 1: col3 -> Rcol3
- y1 pad 1: col6 -> Lcol6
- z1 pad 1: col2 -> Rcol2
- |1 pad 1: col13 -> Lcol13
Routing:
- net row2: vias 1 -> 0
- net row1: vias 2 -> 0
- net col9: vias 1 -> 0
- net col5: vias 1 -> 0
- net Net-(U1-PadRST): vias 1 -> 0
- net Net-(;1-Pad2): vias 0 -> 1

Commit message: とりあえず回路図はできたかな
Parts:
- AltL1, AltR1: footprint keyboard:Hybrid_Plate_125H -> keyboard:Hybrid_Plate_100H
- moved U1 375.1 mm to (-61.0, 234.9)
- moved U2 345.2 mm to (463.6, 143.5)
- moved J2 273.2 mm to (313.7, 189.2)
- moved J1 258.9 mm to (-3.81, 229.9)
- moved s3 255.4 mm to (322.6, 170.2)
- moved p2 251.4 mm to (-1.27, 212.1)
- moved s2 251.1 mm to (-15.2, 208.3)
- moved p3 211.6 mm to (256.5, 175.3)
- moved D29 123.1 mm to (151.1, 142.2)
- moved D51 121.9 mm to (163.8, 177.8)
- moved D61 102.0 mm to (229.9, 200.7)
- moved SP1 7.51 mm to (31.9, 129.5)
- moved winL1 3.14 mm to (-8.64, 129.5)
- moved AltL1 2.17 mm to (-32.5, 129.5)
- moved d1 1.52 mm to (10.2, 91.4)
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
Commit message: ちょっと前にスイッチの街がとかを修正したやつ
Parts:
- AltL1, AltR1: footprint keyboard:Hybrid_Plate_100H -> keyboard:MX_PCB_100H
- BackSP1: footprint keyboard:Hybrid_Plate_150H -> keyboard:MX_PCB_150H
- Control1: footprint keyboard:Hybrid_Plate_175H -> keyboard:MX_PCB_175H
- D61: footprint keyboard:Diode -> keyboard:Diode-dual
- ESC1, Fn1, L1, e1, f1, g1, h1, i1, j1, k1, m1, n1, o1, p1, q1, r1, s1: footprint keyboard:Hybrid_PCB_100H -> keyboard:MX_PCB_100H
- Enter1: footprint keyboard:Hybrid_PCB_225H -> keyboard:MX_PCB_225H
- SP2: footprint keyboard:MX_Plate_225H -> keyboard:MX_PCB_275H
- U1: moved to F.Cu
- U2: moved to B.Cu
- sharp1, t1, u1, v1, w1, x1, y1, z1, |1: footprint keyboard:MX_Plate_100H -> keyboard:MX_PCB_100H
- shiftL1: footprint keyboard:Hybrid_Plate_225H -> keyboard:MX_PCB_225H
- shiftR1: footprint keyboard:Hybrid_Plate_275H -> keyboard:MX_PCB_175H
- tab1: footprint keyboard:Hybrid_PCB_150H -> keyboard:MX_PCB_150H
- winL1, winR1: footprint keyboard:MX_Plate_150H -> keyboard:MX_PCB_100H
- moved U2 251.3 mm to (212.9, 126.4)
- moved D49 214.9 mm to (154.8, 51.1), turned to 270 degrees
- moved J1 199.9 mm to (-76.1, 43.5)
- moved D50 197.4 mm to (166.2, 70.4), turned to 270 degrees
- moved J2 165.4 mm to (234.9, 43.8)
- moved D48 141.4 mm to (145.1, 127.0), turned to 270 degrees
- moved D61 137.1 mm to (114.9, 126.0), turned to 270 degrees
- moved p2 130.8 mm to (-43.6, 88.3)
- moved D44 124.4 mm to (137.0, 52.3), turned to 270 degrees
- moved D54 114.5 mm to (176.4, 52.3), turned to 270 degrees
- moved p3 114.4 mm to (188.7, 83.1)
- moved s2 110.5 mm to (-74.6, 115.1), turned to 90 degrees
- moved D29 109.7 mm to (68.5, 70.1), turned to 270 degrees
- moved D36 107.6 mm to (106.6, 70.1), turned to 270 degrees
- moved s3 107.1 mm to (233.0, 111.5), turned to 270 degrees
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Routing:
- net row4: vias 1 -> 0
- net col3: vias 1 -> 0
- net col10: vias 1 -> 0
